File: BLDC_controller_0.sch (EAGLE design)
At the start: 32 parts, among them IC1 78L05Z

Commit message: Add files via upload
Parts:
- added C12, C18, C20, C22, C23, C24, C25, C26: 10nF, rcl:C-EU025-024X044
- added C17, C19, C21: 47uF, rcl:CPOL-EUE5-10.5
- added C27, C28, C29: 100nF, rcl:C-EU025-024X044
- added D1, D2, D4, D5, D7, D8: 1N4004, diode:1N4004
- added HALL: (no value), con-amp-mt:S05P
- added LED1: LAP4-BOTTOM, led:LAP4-BOTTOM
- added MOTOR: (no value), con-amp-mt:S03P
- added Q10, Q11, Q12, Q7, Q8, Q9: IRF540, transistor-power:IRF540
- added R10, R17, R2, R25, R30, R31, R35, R36, R40, R41, R44, R45, R46, R47, R49, R5, R9: 2.2k, rcl:R-EU_0204/5
- added R11, R26, R29, R34, R39, R6: 510E, rcl:R-EU_0204/5
- added R12, R27, R32, R37, R42, R7: 100E, rcl:R-EU_0204/5
- added R16, R28, R8: 202k, rcl:R-EU_0204/5
- added R33, R38, R43: 10k, rcl:R-EU_0204/5
- added R48: 9.4k, rcl:R-EU_0204/5
- added R50: 1.2k, rcl:R-EU_0204/5
- added R51: 220E, rcl:R-EU_0204/5
- added SUPPLY_MAIN, THROTTLE: (no value), con-amp-mt:S02P
- added T10, T13, T16, T19, T2, T4, T5, T7, T8: (no value), transistor-neu-to92:2N3906-PNP-TO92-EBC
- added T11, T12, T14, T15, T17, T18, T3, T6, T9: 2N3904, transistor:2N3904
- added U$1: D79F9211DF9F9211, D79F9211:D79F9211DF9F9211
Connections:
- removed net N$2 (its old number): C11.1, R18.2, R19.2, R20.2
- new net +15V: C3.1, C4.1, C5.1, D2.A, D5.A, D8.A, LM317.OUT, R14.1, R29.2, R34.2, R39.2, R4.2, T13.E, T16.E, T19.E
- new net MOTOR_U: C12.2, C17.-, C18.2, C19.-, C20.2, C21.-, MOTOR-1.S, MOTOR-2.S, MOTOR-3.S, Q10.S, Q11.S, Q12.S, Q7.D, Q8.D, Q9.D, R10.1, R25.1, R33.2, R38.2, R43.2, R5.1, T10.C, T4.C, T7.C
- new net N$1: R30.2, T11.E
- new net N$10: R2.2, T3.E
- new net N$19: R8.1, U$1.P10
- new net N$20: R6.1, T2.B, T3.C
- new net N$21: R8.2, T3.B
- new net N$22: D1.A, R5.2, T2.C, T4.B
- new net N$23: D1.C, R7.2
- new net N$24: C12.1, Q12.G, R7.1, T4.E
- new net N$25: C17.+, D2.C, R6.2, T2.E
- new net N$27: R9.2, T6.E
- new net N$28: R32.2, T13.C
- new net N$29: R11.1, T5.B, T6.C
- new net N$30: C28.1, R48.1, R49.1, R50.2
- new net N$31: R16.2, T6.B
- new net N$32: D4.A, R10.2, T5.C, T7.B
- new net N$33: D4.C, R12.2
- new net N$34: C18.1, Q11.G, R12.1, T7.E
- new net N$35: C19.+, D5.C, R11.2, T5.E
- new net N$36: R40.2, T17.E
- new net N$37: R16.1, U$1.P12
- new net N$39: R17.2, T9.E
- new net N$40: R26.1, T8.B, T9.C
- new net N$41: R28.2, T9.B
- new net N$42: D7.A, R25.2, T10.B, T8.C
- new net N$43: D7.C, R27.2
- new net N$44: C20.1, Q10.G, R27.1, T10.E
- new net N$45: C21.+, D8.C, R26.2, T8.E
- new net N$46: C22.1, Q7.G, R32.1, T12.C
- new net N$47: R28.1, U$1.P50
- new net N$49: R29.1, T11.C, T13.B
- new net N$50: R37.2, T16.C
- new net N$51: R30.1, R31.2, U$1.P83
- new net N$52: R31.1, T12.B
- new net N$53: C25.1, LED1.C, R44.1, U$1.P22
- new net N$54: R42.2, T19.C
- new net N$55: C23.1, Q8.G, R37.1, T15.C
- new net N$56: R34.1, T14.C, T16.B
- new net N$57: R35.1, R36.2, U$1.P13
- new net N$58: R36.1, T15.B
- new net N$59: C22.2, C23.2, C24.2, Q7.S, Q8.S, Q9.S, R33.1, R38.1, R43.1, R44.2, R45.2, R46.2
- new net N$60: C26.1, R46.1, R47.1, U$1.P80
- new net N$61: C24.1, Q9.G, R42.1, T18.C
- new net N$62: R39.1, T17.C, T19.B
- new net N$63: R40.1, R41.2, U$1.P51
- new net N$64: R41.1, T18.B
- new net N$65: R49.2, U$1.P151
- new net N$66: LED1.A, U$1.P20
- new net N$67: R51.2
- new net N$68: C29.2, U$1.REGC
- new net VPP1: THROTTLE-1.S, U$1.P150
- net +5V: now also C11.1, C16.+, C27.2, C6.1, C7.1, IC1.VO, R18.2, R19.2, R20.2, R47.2, T11.B, T14.B, T17.B, U$1.AVREF, U$1.RESET_BAR, U$1.VDD; no longer C3.1, C4.1, C5.1, LM317.OUT, R14.1, R4.2
- net 0V: now also C25.2, C26.2, C27.1, C28.2, C29.1, HALL-5.S, R17.1, R2.1, R45.1, R50.1, R51.1, R9.1, SUPPLY_MAIN-2.S, T12.E, T15.E, T18.E, THROTTLE-2.S, U$1.AVSS, U$1.VSS
- net N$11: now also U$1.P121/X1
- net N$12: now also U$1.P122
- net N$14: now also HALL-1.S
- net N$15: now also U$1.P32
- net N$17: now also U$1.P74
- net N$18: now also U$1.P120
- net N$3: now also HALL-2.S
- net N$7: now also R35.2, T14.E; no longer C16.+, C6.1, C7.1, IC1.VO
- net N$8: now also HALL-3.S
- net N$9: now also HALL-4.S
- net VPP: now also Q10.D, Q11.D, Q12.D, R48.2, SUPPLY_MAIN-1.S
Other:
- note added: "15/14V"
- note added: "38/36V"
- note added: "5V"
- note added: "CPU-14"
- note added: "CPU-16"
- note added: "CPU-22"
- note added: "CPU-23"
- note added: "CPU-24"
- note added: "CPU-25"
- note added: "CPU-27"
- note added: "CPU-28"
- note added: "CPU-31"
- note added: "CPU-41"
- note added: "CPU-44"
- note added: "CPU-7"
- note added: "CPU-8"
- note added: "H+"
- note added: "MOTOR_W"
- note added: "MOTOR_v"
- note added: "U"
- note added: "V"
- note added: "W"
- note added: "gnd"
- note removed: "50mA"
- moved on the sheet: C10, C11, C8, C9, R15, R18, R19, R20, R21, R22, R23, R24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

Commit message: Add files via upload
final bldc_motor_controller
Parts:
- added C30, C32, C34, C36, C38, C40: 10nF, rcl:C-EU025-024X044
- added C31, C33, C35, C37, C39, C41: 47uF, rcl:CPOL-EUE5-10.5
- added D10, D11, D12, D13, D14, D15, D16, D17, D18, D3, D6, D9: 1N4004, diode:1N4004
- added IC2: LM393D, linear:LM393D
- added LED2: LAP4-BOTTOM, led:LAP4-BOTTOM
- added Q1, Q2, Q3, Q4, Q5, Q6: IRF540, transistor-power:IRF540
- added R52, R53, R57, R58, R62, R63, R67, R68, R72, R73, R77, R78, R82, R83: 2.2k, rcl:R-EU_0204/5
- added R54, R59, R64, R69, R74, R79: 510E, rcl:R-EU_0204/5
- added R55, R60, R65, R70, R75, R80: 100E, rcl:R-EU_0204/5
- added R56, R61, R66, R71, R76, R81: 202k, rcl:R-EU_0204/5
- added R84: 3.3k, rcl:R-EU_0204/5
- added T20, T22, T23, T25, T26, T28, T29, T31, T32, T34, T35, T37: (no value), transistor-neu-to92:2N3906-PNP-TO92-EBC
- added T21, T24, T27, T30, T33, T36: 2N3904, transistor:2N3904
Connections:
- new net N$101: R72.2, T33.E
- new net N$102: R74.1, T32.B, T33.C
- new net N$103: R76.2, T33.B
- new net N$104: D15.A, R73.2, T32.C, T34.B
- new net N$105: D15.C, R75.2
- new net N$106: C38.1, Q5.G, R75.1, T34.E
- new net N$107: C39.+, D16.C, R74.2, T32.E
- new net N$109: R77.2, T36.E
- new net N$110: R79.1, T35.B, T36.C
- new net N$111: R81.2, T36.B
- new net N$112: D17.A, R78.2, T35.C, T37.B
- new net N$113: D17.C, R80.2
- new net N$114: C40.1, Q6.G, R80.1, T37.E
- new net N$115: C41.+, D18.C, R79.2, T35.E
- new net N$117: R61.1, U$1.P30
- new net N$118: R71.1, U$1.P31
- new net N$119: R81.1, U$1.P71
- new net N$120: R76.1, U$1.P72
- new net N$121: R66.1, U$1.P70
- new net N$122: R56.1, U$1.P52
- new net N$123: IC2A.OUT, IC2B.+IN
- new net N$124: IC2A.-IN, IC2B.-IN, R82.2, R83.1
- new net N$125: LED2.C, R84.1
- new net N$126: IC2B.OUT, LED2.A
- new net N$19: R57.2, T24.E
- new net N$69: R52.2, T21.E
- new net N$70: R54.1, T20.B, T21.C
- new net N$71: R56.2, T21.B
- new net N$72: D3.A, R53.2, T20.C, T22.B
- new net N$73: D3.C, R55.2
- new net N$74: C30.1, Q1.G, R55.1, T22.E
- new net N$75: C31.+, D6.C, R54.2, T20.E
- new net N$78: R59.1, T23.B, T24.C
- new net N$79: R61.2, T24.B
- new net N$80: D9.A, R58.2, T23.C, T25.B
- new net N$81: D9.C, R60.2
- new net N$82: C32.1, Q2.G, R60.1, T25.E
- new net N$83: C33.+, D10.C, R59.2, T23.E
- new net N$85: R62.2, T27.E
- new net N$86: R64.1, T26.B, T27.C
- new net N$87: R66.2, T27.B
- new net N$88: D11.A, R63.2, T26.C, T28.B
- new net N$89: D11.C, R65.2
- new net N$90: C34.1, Q3.G, R65.1, T28.E
- new net N$91: C35.+, D12.C, R64.2, T26.E
- new net N$93: R67.2, T30.E
- new net N$94: R69.1, T29.B, T30.C
- new net N$95: R71.2, T30.B
- new net N$96: D13.A, R68.2, T29.C, T31.B
- new net N$97: D13.C, R70.2
- new net N$98: C36.1, Q4.G, R70.1, T31.E
- new net N$99: C37.+, D14.C, R69.2, T29.E
- net +15V: now also D10.A, D12.A, D14.A, D16.A, D18.A, D6.A
- net +5V: now also R83.2
- net 0V: now also IC2A.+IN, R52.1, R57.1, R62.1, R67.1, R72.1, R77.1, R82.1, R84.2
- net MOTOR_U: now also C30.2, C31.-, C32.2, C33.-, C34.2, C35.-, C36.2, C37.-, C38.2, C39.-, C40.2, C41.-, Q1.S, Q2.S, Q3.S, Q4.S, Q5.S, Q6.S, R53.1, R58.1, R63.1, R68.1, R73.1, R78.1, T22.C, T25.C, T28.C, T31.C, T34.C, T37.C
- net VPP: now also Q1.D, Q2.D, Q3.D, Q4.D, Q5.D, Q6.D
